File: cool-keyboard.kicad_pcb (KiCad board)
At the start: 2 copper layers, 81.8 x 81 mm, 22 parts, among them SW1 SW_Push_45deg, SW10 SW_Push_45deg, SW13 RotaryEncoder_Switch, SW2 SW_Push_45deg, SW3 SW_Push_45deg, SW4 SW_Push_45deg, SW5 SW_Push_45deg, SW6 SW_Push_45deg, SW7 SW_Push_45deg, SW8 SW_Push_45deg, SW9 SW_Push_45deg, U2 MOUDLE-SEEEDUINO-XIAO

Commit message: traces
Routing:
- net COL2: track 0.00 -> 96.6 mm
- net COL3: track 0.00 -> 90.3 mm
- net COL1: track 0.00 -> 80.8 mm
- net GND: track 0.00 -> 59.9 mm
- net EC11SW: track 0.00 -> 59.5 mm
- net ROW1: track 0.00 -> 52.0 mm
- net COL0: track 0.00 -> 48.9 mm
- net Net-(D10-A): track 0.00 -> 48.1 mm
- net Net-(D9-A): track 0.00 -> 47.3 mm
- net Net-(D5-A): track 0.00 -> 46.2 mm
- net EC11A: track 0.00 -> 45.6 mm
- net EC11B: track 0.00 -> 42.9 mm
- net ROW2: track 0.00 -> 39.7 mm
- net Net-(D4-A): track 0.00 -> 39.1 mm
- net Net-(D8-A): track 0.00 -> 37.4 mm
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