File: cool-keyboard.kicad_sch (KiCad schematic)
At the start: 33 parts, among them U1 MOUDLE-SEEEDUINO-XIAO

Commit message: finish sch + basic pcb
Parts:
- removed D1, D10, D11, D12, D13, D14, D15, D16, D2, D3, D4, D5, D6, D7, D8, D9: D_Small, Diode_SMD:D_SOD-123, symbol Device:D_Small
- removed MX1, MX10, MX11, MX12, MX13, MX14, MX15, MX16, MX2, MX3, MX4, MX5, MX6, MX7, MX8, MX9: MX-NoLED, MX_Alps_Hybrid:MX-1U-NoLED, symbol MX_Alps_Hybrid:MX-NoLED
- removed U1: MOUDLE-SEEEDUINO-XIAO, XIAO_PCB:MOUDLE14P-2.54-21X17.8MM, symbol MOUDLE-SEEEDUINO-XIAO:MOUDLE-SEEEDUINO-XIAO
- added D1, D10, D2, D3, D4, D5, D6, D7, D8, D9: D, Diode_THT:D_5KP_P10.16mm_Horizontal, symbol Device:D
- added SW1, SW10, SW2, SW3, SW4, SW5, SW6, SW7, SW8, SW9: SW_Push_45deg, MX_Solderable:MX-Solderable-1U, symbol Switch:SW_Push_45deg
- added SW13: RotaryEncoder_Switch, Rotary_Encoder:RotaryEncoder_Alps_EC11E-Switch_Vertical_H20mm, symbol Device:RotaryEncoder_Switch
- added U2: MOUDLE-SEEEDUINO-XIAO, XIAO_PCB:MOUDLE14P-2.54-21X17.8MM, symbol MOUDLE-SEEEDUINO-XIAO:MOUDLE-SEEEDUINO-XIAO
Connections:
- net +5V: now also U2.14 (5V)
- net COL0: now also SW1.1, SW5.1, U2.1 (PA02_A0_D0)
- net COL1: now also SW2.1, SW6.1, SW9.1, U2.2 (PA4_A1_D1)
- net COL2: now also SW10.1, SW3.1, SW7.1, U2.3 (PA10_A2_D2)
- net COL3: now also SW4.1, SW8.1, U2.4 (PA11_A3_D3)
- net GND: now also SW13.C, SW13.S1, U2.13 (GND)
- net ROW0: now also D1.1 (K), D2.1 (K), D3.1 (K), D4.1 (K), U2.5 (PA8_A4_D4_SDA)
- net ROW1: now also D5.1 (K), D6.1 (K), D7.1 (K), D8.1 (K), U2.6 (PA9_A5_D5_SCL)
- net ROW2: now also D10.1 (K), D9.1 (K), U2.7 (PB08_A6_D6_TX)
- new net: D2.2 (A), SW2.2
- new net: D7.2 (A), SW7.2
- new net: D8.2 (A), SW8.2
- new net: D4.2 (A), SW4.2
- new net: D1.2 (A), SW1.2
- new net: D3.2 (A), SW3.2
- new net: D6.2 (A), SW6.2
- new net: D9.2 (A), SW9.2
- new net: D10.2 (A), SW10.2
- new net: D5.2 (A), SW5.2
- new net EC11A: SW13.A, U2.9 (PA7_A8_D8_SCK)
- new net EC11B: SW13.B, U2.11 (PA6_A10_D10_MOSI)
- new net EC11SW: SW13.S2, U2.10 (PA5_A9_D9_MISO)

Commit message: add ssd1306
Parts:
- removed SW13: RotaryEncoder_Switch, Rotary_Encoder:RotaryEncoder_Alps_EC11E-Switch_Vertical_H20mm, symbol Device:RotaryEncoder_Switch
- added Brd1: SSD1306, SSD1306:128x64OLED, symbol SSD1306-128x64_OLED:SSD1306
- D1, D10, D2, D3, D4, D5, D6, D7, D8, D9: footprint Diode_THT:D_5KP_P10.16mm_Horizontal -> Diode_THT:D_A-405_P10.16mm_Horizontal
Connections:
- net EC11A is gone; now on net ROW1: U2.9 (PA7_A8_D8_SCK)
- net EC11SW is gone; now on net ROW2: U2.10 (PA5_A9_D9_MISO)
- net GND: now also Brd1.1 (GND)
- net ROW0: now also U2.8 (PB09_A7_D7_RX); no longer U2.5 (PA8_A4_D4_SDA)
- net ROW1: no longer U2.6 (PA9_A5_D5_SCL)
- net ROW2: no longer U2.7 (PB08_A6_D6_TX)
- net SCR3V3: now reaches U2.12 (3V3)
- net SCR3V3: now also Brd1.2 (VCC)
- net EC11B: no longer names the net of U2.11 (PA6_A10_D10_MOSI)
- new net: Brd1.3 (SCL), U2.6 (PA9_A5_D5_SCL)
- new net: Brd1.4 (SDA), U2.5 (PA8_A4_D4_SDA)
